File: HydroB V2_SubBoard/_autosave-Power supply.kicad_sch (KiCad schematic)
At the start: 14 parts, among them U4 LMR33620ADDA

Commit message: PCB update finalize
Connections:
- net A: no longer names the net of C24.2, L2.1, U4.8 (SW)
Changed lines of the file:
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@@
-		)
-	)
-	(global_label "A"
-		(shape input)
-		(at 146.05 100.33 90)
-		(fields_autoplaced yes)
-		(effects
-			(font
-				(size 1.27 1.27)
-			)
-			(justify left)
-		)
-		(property "Intersheetrefs" "${INTERSHEET_REFS}"
-			(at 146.05 96.2562 90)
-			(effects
-				(font
-					(size 1.27 1.27)
-				)
-				(justify left)
-				(hide yes)
-			)
 		)
 	)
