File: HydroB V2_SubBoard/HydroB V2.kicad_pcb (KiCad board)
At the start: 4 copper layers, 180.2 x 120 mm, 132 parts, among them J1 Conn_01x02_Pin, J10 Screw_Terminal_01x02, J16 Screw_Terminal_01x02, J2 12V, J3 Screw_Terminal_01x02, J4 Conn_01x04_Pin, J5 Conn_01x02_Pin, J6 SENSOR, J7 Conn_01x02_Pin, J8 Screw_Terminal_01x02, J9 Screw_Terminal_01x02, Q1 S8050, Q2 S8050, Q3 S8050, Q4 S8050, Q5 S8050, Q6 S8050, Q7 S8050, SW1 SW_Push, U1 STM32F103C8Tx, U11 PC817, U12 PC817, U13 PC817, U2 PC817, U3 SN65HVD72DR, U4 LMR33620ADDA, U5 PC817, Y1 8Mhz

Commit message: PCB placement
Parts:
- removed D16, D17, D7, D8: LED_Small, LED_SMD:LED_0805_2012Metric
- removed R28: 1K, Resistor_SMD:R_0603_1608Metric
- removed R30: 1k, Resistor_SMD:R_0603_1608Metric
- removed kibuzzard-66A86A88 (x3): G***, kibuzzard-66A86A88
- removed kibuzzard-66A86AEA: G***, kibuzzard-66A86AEA
- removed kibuzzard-66A86B8E (x3): G***, kibuzzard-66A86B8E
- removed kibuzzard-66A86BAD: G***, kibuzzard-66A86BAD
- removed kibuzzard-66A86BBB: G***, kibuzzard-66A86BBB
- removed kibuzzard-66A8B27E: G***, kibuzzard-66A8B27E
- removed kibuzzard-66A8B2A7: G***, kibuzzard-66A8B2A7
- removed kibuzzard-66AAEFF5 (x5): G***, kibuzzard-66AAEFF5
- removed kibuzzard-66AAF0AE: G***, kibuzzard-66AAF0AE
- removed kibuzzard-66AAF0BB: G***, kibuzzard-66AAF0BB
- removed kibuzzard-66AAF0C8: G***, kibuzzard-66AAF0C8
- removed kibuzzard-66AAF0D5: G***, kibuzzard-66AAF0D5
- removed kibuzzard-66AAF0E0: G***, kibuzzard-66AAF0E0
- removed kibuzzard-66AAF0E8: G***, kibuzzard-66AAF0E8
- removed kibuzzard-66AAF2E3: G***, kibuzzard-66AAF2E3
- added J11: Conn_01x02_Pin, Connector_PinHeader_2.00mm:PinHeader_1x02_P2.00mm_Vertical, F.Cu at (214.6, 56.9)
- added J12: Conn_01x02_Pin, Connector_PinHeader_2.00mm:PinHeader_1x02_P2.00mm_Vertical, F.Cu at (208.6, 76.8)
- added TP1: TestPoint, TestPoint:TestPoint_Loop_D1.80mm_Drill1.0mm_Beaded, F.Cu at (191.7, 88.5)
- added TP2: TestPoint, TestPoint:TestPoint_Loop_D1.80mm_Drill1.0mm_Beaded, F.Cu at (191.7, 83.7)
- added TP3: TestPoint, TestPoint:TestPoint_Loop_D1.80mm_Drill1.0mm_Beaded, F.Cu at (220.8, 71.4)
- added TP4: TestPoint, TestPoint:TestPoint_Loop_D1.80mm_Drill1.0mm_Beaded, F.Cu at (220.8, 76.2)
- added kibuzzard-66AB40EF: G***, kibuzzard-66AB40EF, F.Cu at (97.3, 35.4)
- added kibuzzard-66AB40EF: G***, kibuzzard-66AB40EF, F.Cu at (189.7, 35.4)
- added kibuzzard-66AB40EF: G***, kibuzzard-66AB40EF, F.Cu at (75.5, 35.4)
- added kibuzzard-66AB40EF: G***, kibuzzard-66AB40EF, F.Cu at (205.6, 36.1)
- added kibuzzard-66AB40EF: G***, kibuzzard-66AB40EF, F.Cu at (141.1, 35.4)
- added kibuzzard-66AB40EF: G***, kibuzzard-66AB40EF, F.Cu at (176.9, 35.4)
- added kibuzzard-66AB40EF: G***, kibuzzard-66AB40EF, F.Cu at (119.2, 35.4)
- added kibuzzard-66AB40EF: G***, kibuzzard-66AB40EF, F.Cu at (163.0, 35.4)
- added kibuzzard-66AB4112: G***, kibuzzard-66AB4112, F.Cu at (94.8, 35.4)
- added kibuzzard-66AB4112: G***, kibuzzard-66AB4112, F.Cu at (160.5, 35.4)
- added kibuzzard-66AB4112: G***, kibuzzard-66AB4112, F.Cu at (116.7, 35.4)
- added kibuzzard-66AB4112: G***, kibuzzard-66AB4112, F.Cu at (73.0, 35.4)
- added kibuzzard-66AB4112: G***, kibuzzard-66AB4112, F.Cu at (138.6, 35.4)
- added kibuzzard-66AB4A9F: G***, kibuzzard-66AB4A9F, F.Cu at (187.2, 35.4)
- added kibuzzard-66AB4A9F: G***, kibuzzard-66AB4A9F, F.Cu at (174.4, 35.4)
- added kibuzzard-66AB4A9F: G***, kibuzzard-66AB4A9F, F.Cu at (203.6, 36.1)
- added kibuzzard-66AB4C8A: G***, kibuzzard-66AB4C8A, F.Cu at (201.6, 36.1)
- added kibuzzard-66AB4C8F: G***, kibuzzard-66AB4C8F, F.Cu at (199.6, 36.1)
- C14, C15: value 22PF -> 22pF
- R17, R21: value 10k -> Variable Resistor
- R24, R25, R26, R27: value 1K -> 445R
- R29: value 1k -> 445R
- moved J6 153.8 mm to (67.1, 93.3), turned to 90 degrees
- moved R29 83.4 mm to (98.2, 47.3), turned to 180 degrees
- moved J10 60.4 mm to (160.4, 40.4), turned to 0 degrees
- moved R25 57.7 mm to (142.0, 47.4), turned to 180 degrees
- moved R39 53.1 mm to (166.0, 81.0), turned to 180 degrees
- moved U13 50.5 mm to (159.2, 81.1), turned to 90 degrees
- moved J8 49.0 mm to (116.7, 40.4), turned to 0 degrees
- moved J16 48.4 mm to (94.8, 40.4), turned to 0 degrees
- moved J3 47.9 mm to (73.0, 40.4), turned to 0 degrees
- moved J9 47.5 mm to (138.5, 40.4), turned to 0 degrees
- moved R14 45.9 mm to (166.0, 78.8), turned to 0 degrees
- moved C13 45.6 mm to (189.1, 98.3), turned to 180 degrees
- moved Q4 44.8 mm to (166.0, 71.7), turned to 90 degrees
- moved R23 43.2 mm to (166.0, 76.5)
- moved R21 42.7 mm to (173.1, 48.9), turned to 90 degrees
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Connections:
- C25 pad 1: +3.3V -> Net-(J12-Pin_1)
- C26 pad 1: +3.3V -> Net-(J12-Pin_1)
- C27 pad 1: +3.3V -> Net-(J12-Pin_1)
- C28 pad 1: +3.3V -> Net-(J12-Pin_1)
- C29 pad 1: +3.3V -> Net-(J12-Pin_1)
- D11 pad 2: Net-(D10-A) -> Net-(D11-A)
- D3 pad 2: Net-(D12-A) -> Net-(D3-A)
- D5 pad 2: Net-(D13-A) -> Net-(D5-A)
- D6 pad 2: Net-(D14-A) -> Net-(D6-A)
- D9 pad 2: Net-(D2-A) -> Net-(D9-A)
- J10 pad 1: Net-(J10-Pin_1) -> Net-(D14-A)
- J16 pad 1: Net-(J16-Pin_1) -> Net-(D11-A)
- J2 pad 1: +12V -> Net-(J11-Pin_1)
- J3 pad 1: Net-(J3-Pin_1) -> Net-(D9-A)
- J5 pad 1: +3.3V -> Net-(J5-Pin_1)
- J7 pad 1: +3.3V -> Net-(J7-Pin_1)
- J8 pad 1: Net-(J8-Pin_1) -> Net-(D12-A)
- J9 pad 1: Net-(J9-Pin_1) -> Net-(D13-A)
- L2 pad 2: +3.3V -> Net-(J12-Pin_1)
- Q2 pad 3: Net-(D12-A) -> Net-(D3-A)
- Q3 pad 3: Net-(D13-A) -> Net-(D5-A)
- Q4 pad 3: Net-(D14-A) -> Net-(D6-A)
- R17 pad 1: /HydroB/Block Sensor1/RS485_TX -> +3.3V
- R17 pad 2: Net-(D8-K) -> Net-(J5-Pin_1)
- R21 pad 1: /HydroB/Block Sensor1/RS485_RX -> +3.3V
- R21 pad 2: Net-(D7-K) -> Net-(J7-Pin_1)
- R25 pad 2: Net-(D11-K) -> Net-(D13-K)
- R27 pad 1: +3.3V -> GND
- R27 pad 2: Net-(D13-K) -> Net-(D14-K)
- R29 pad 1: SWCLK -> +3.3V
- R29 pad 2: Net-(D16-A) -> Net-(D11-K)
- R7 pad 2: +3.3V -> Net-(J12-Pin_1)
- U10 pad 1: Net-(J10-Pin_1) -> Net-(D14-A)
- U10 pad 2: Net-(J10-Pin_1) -> Net-(D14-A)
- U10 pad 3: Net-(D14-A) -> Net-(D6-A)
- U6 pad 1: Net-(J16-Pin_1) -> Net-(D11-A)
- U6 pad 2: Net-(J16-Pin_1) -> Net-(D11-A)
- U7 pad 1: Net-(J3-Pin_1) -> Net-(D9-A)
- U7 pad 2: Net-(J3-Pin_1) -> Net-(D9-A)
- U8 pad 1: Net-(J8-Pin_1) -> Net-(D12-A)
- U8 pad 2: Net-(J8-Pin_1) -> Net-(D12-A)
- U8 pad 3: Net-(D12-A) -> Net-(D3-A)
- U9 pad 1: Net-(J9-Pin_1) -> Net-(D13-A)
- U9 pad 2: Net-(J9-Pin_1) -> Net-(D13-A)
- U9 pad 3: Net-(D13-A) -> Net-(D5-A)
Routing:
- net /HydroB/Block Relay1/RELAY_1: track 135.9 -> 0.00 mm
- net Net-(D15-A1): track 118.1 -> 0.00 mm
- net Net-(D15-A2): track 113.4 -> 0.00 mm
- net /HydroB/Block Relay1/RELAY_2: track 112.4 -> 0.00 mm
- net NRST: track 106.8 -> 0.00 mm, vias 1 -> 0
- net +12V: track 93.1 -> 0.00 mm, vias 57 -> 0
- net /HydroB/Block Relay1/RELAY_3: track 92.0 -> 0.00 mm
- net /HydroB/Block Relay1/RELAY_5: track 73.1 -> 0.00 mm
- net /HydroB/Block Relay1/RELAY_4: track 52.7 -> 0.00 mm
- net SWCLK: track 52.6 -> 0.00 mm, vias 2 -> 0
- net SWDIO: track 47.7 -> 0.00 mm, vias 2 -> 0
- net /HydroB/Block Sensor1/EN_RS485: track 33.6 -> 0.00 mm
- net /HydroB/Block Sensor1/RS485_RX: track 30.9 -> 0.00 mm
- net /HydroB/Block Sensor1/RS485_TX: track 27.9 -> 0.00 mm
- net Net-(D2-A): track 26.6 -> 0.00 mm
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- added copper zone on F.Cu, net (none)
- removed copper zone on F.Cu, net +12V
- removed copper zone on In2.Cu, net +12V
- removed copper zone on F.Cu, net /HydroB/Power Supply1/SW
- removed copper zone on F.Cu, net Net-(U4-FB)
- removed copper zone on F.Cu, net Net-(U4-VCC)
Other:
- outline, holes or cut-outs redrawn

Commit message: PCB placement
Parts:
- removed R18, R2, R22, R23, R3: 10K, Resistor_SMD:R_0603_1608Metric
- added kibuzzard-66AC3E80: G***, kibuzzard-66AC3E80, F.Cu at (217.9, 55.4)
- added kibuzzard-66AC3E8A: G***, kibuzzard-66AC3E8A, F.Cu at (226.7, 90.5)
- added kibuzzard-66AC3EE5: G***, kibuzzard-66AC3EE5, F.Cu at (68.3, 93.3)
- added kibuzzard-66AC3EE5: G***, kibuzzard-66AC3EE5, F.Cu at (222.2, 73.7)
- added kibuzzard-66AC3EFD: G***, kibuzzard-66AC3EFD, F.Cu at (201.3, 72.6)
- added kibuzzard-66AC3F5E: G***, kibuzzard-66AC3F5E, F.Cu at (188.1, 88.5)
- added kibuzzard-66AC3F67: G***, kibuzzard-66AC3F67, F.Cu at (188.1, 83.7)
- added kibuzzard-66AC4019: G***, kibuzzard-66AC4019, F.Cu at (222.1, 94.8)
- added kibuzzard-66AC401E: G***, kibuzzard-66AC401E, F.Cu at (217.3, 94.8)
- D1: footprint LED_SMD:LED_Cree-PLCC4_5x5mm_CW -> LED_SMD:LED_RGB_Wuerth-PLCC4_3.2x2.8mm_150141M173100
- R24, R25, R26, R27, R29: value 445R -> 470R
- R35, R36, R37, R38, R39: value 220R -> 5k
- moved TP3 20.8 mm to (217.3, 91.8), turned to 90 degrees
- moved TP4 15.8 mm to (222.1, 91.8), turned to 90 degrees
- moved D1 1.30 mm to (144.1, 92.5)
- moved R15 0.20 mm to (219.4, 86.0), turned to 180 degrees
Connections:
- R24 pad 1: +3.3V -> GND
- R25 pad 1: +3.3V -> GND
- R26 pad 1: +3.3V -> GND
- R29 pad 1: +3.3V -> GND

Commit message: PCB layout
Parts:
- removed J12: Conn_01x02_Pin, Connector_PinHeader_2.00mm:PinHeader_1x02_P2.00mm_Vertical
- D1: value LED_Small -> Inolux_IN-PI554FCH; footprint LED_SMD:LED_RGB_Wuerth-PLCC4_3.2x2.8mm_150141M173100 -> LED_SMD:LED_Inolux_IN-PI554FCH_PLCC4_5.0x5.0mm_P3.2mm
- moved C9 55.2 mm to (168.8, 87.0), turned to -90 degrees
- moved C10 47.7 mm to (173.2, 83.8), turned to 90 degrees
- moved J11 41.5 mm to (178.2, 77.0), turned to -90 degrees
- moved U4 39.5 mm to (179.1, 85.0), turned to 0 degrees
- moved R8 36.8 mm to (181.3, 89.5), turned to 0 degrees
- moved kibuzzard-66AC3F5E 34.8 mm to (206.9, 59.2)
- moved kibuzzard-66AC3F67 34.0 mm to (211.7, 59.2)
- moved R7 30.3 mm to (185.4, 89.5), turned to 0 degrees
- moved C24 30.2 mm to (185.1, 83.8), turned to 90 degrees
- moved TP1 29.7 mm to (206.8, 63.0), turned to -90 degrees
- moved L2 29.7 mm to (188.6, 78.8)
- moved C25 29.6 mm to (185.6, 87.5), turned to 180 degrees
- moved TP2 28.8 mm to (211.7, 63.0), turned to -90 degrees
- moved R34 28.4 mm to (202.2, 52.2), turned to 180 degrees
- moved C13 27.8 mm to (197.7, 71.8), turned to 90 degrees
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Connections:
- C25 pad 1: Net-(J12-Pin_1) -> +3.3V
- C26 pad 1: Net-(J12-Pin_1) -> +3.3V
- C27 pad 1: Net-(J12-Pin_1) -> +3.3V
- C28 pad 1: Net-(J12-Pin_1) -> +3.3V
- C29 pad 1: Net-(J12-Pin_1) -> +3.3V
- D1 pad 1: GND -> unconnected-(D1-VSS-Pad1)
- D1 pad 2: Net-(D1-A) -> unconnected-(D1-DIN-Pad2)
- D1 pad 3: (no net) -> unconnected-(D1-VDD-Pad3)
- D1 pad 4: (no net) -> unconnected-(D1-DO-Pad4)
- L2 pad 2: Net-(J12-Pin_1) -> +3.3V
- R1 pad 2: Net-(D1-A) -> unconnected-(R1-Pad2)
- R7 pad 2: Net-(J12-Pin_1) -> +3.3V
- U1 pad 11: unconnected-(U1-PA1-Pad11) -> /HydroB/Block Sensor1/EN_RS485
- U1 pad 14: /HydroB/Block Sensor1/EN_RS485 -> unconnected-(U1-PA4-Pad14)
- U1 pad 18: unconnected-(U1-PB0-Pad18) -> LED1
- U1 pad 21: unconnected-(U1-PB10-Pad21) -> LED2
- U1 pad 30: LED1 -> unconnected-(U1-PA9-Pad30)
- U1 pad 32: LED2 -> unconnected-(U1-PA11-Pad32)
- U1 pad 39: unconnected-(U1-PB3-Pad39) -> /HydroB/Block Relay1/RELAY_1
- U1 pad 41: /HydroB/Block Relay1/RELAY_4 -> /HydroB/Block Relay1/RELAY_2
- U1 pad 42: /HydroB/Block Relay1/RELAY_5 -> /HydroB/Block Relay1/RELAY_3
- U1 pad 43: /HydroB/Block Relay1/RELAY_3 -> unconnected-(U1-PB7-Pad43)
- U1 pad 45: /HydroB/Block Relay1/RELAY_2 -> /HydroB/Block Relay1/RELAY_4
- U1 pad 46: /HydroB/Block Relay1/RELAY_1 -> /HydroB/Block Relay1/RELAY_5
Routing:
- net Net-(D15-A1): track 0.00 -> 232.0 mm
- net Net-(D15-A2): track 0.00 -> 228.1 mm
- net /HydroB/Block Relay1/RELAY_1: track 0.00 -> 124.8 mm
- net /HydroB/Block Relay1/RELAY_2: track 0.00 -> 101.4 mm
- net NRST: track 0.00 -> 81.1 mm
- net /HydroB/Block Relay1/RELAY_3: track 0.00 -> 78.6 mm
- net /HydroB/Block Relay1/RELAY_4: track 0.00 -> 52.8 mm
- net LED: track 0.00 -> 51.9 mm
- net /HydroB/Block Relay1/RELAY_5: track 0.00 -> 31.6 mm
- net /HydroB/Block Sensor1/EN_RS485: track 0.00 -> 27.9 mm
- net /HydroB/Block Sensor1/RS485_TX: track 0.00 -> 27.9 mm
- net LED1: track 0.00 -> 23.5 mm
- net /HydroB/Block Sensor1/RS485_RX: track 0.00 -> 23.4 mm
- net Net-(D9-A): track 0.00 -> 20.4 mm
- net Net-(D11-A): track 0.00 -> 20.4 mm
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- added copper zone on F.Cu, net +12V
- added copper zone on In1.Cu, net +12V
- added copper zone on F.Cu, net /HydroB/Power Supply1/SW
- added copper zone on In1.Cu, net Net-(J11-Pin_1)
- added copper zone on F.Cu, net Net-(U4-FB)
- removed copper zone on F.Cu, net (none)

Commit message: PCB layout
Routing:
- net GND: vias 731 -> 763
- net +3.3V: vias 60 -> 48
- net +12V: vias 70 -> 50
