File: HydroB V2_SubBoard/HydroB V2.kicad_pcb (KiCad board)
At the start: 4 copper layers, 180.2 x 120 mm, 130 parts, among them J1 Conn_01x02_Pin, J10 Screw_Terminal_01x02, J11 Conn_01x02_Pin, J16 Screw_Terminal_01x02, J2 12V, J3 Screw_Terminal_01x02, J4 Conn_01x04_Pin, J5 Conn_01x02_Pin, J6 SENSOR, J7 Conn_01x02_Pin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

Commit message: update
Parts:
- added D7: LED_Small, LED_SMD:LED_0805_2012Metric, F.Cu at (148.1, 95.3)
- added Q8: S8050, Package_TO_SOT_SMD:SOT-23, F.Cu at (145.0, 91.7)
- added R18: 10K, Resistor_SMD:R_0603_1608Metric, F.Cu at (144.0, 87.8)
- added R2: 2k, Resistor_SMD:R_0603_1608Metric, F.Cu at (142.1, 97.5)
- added R3: 1K, Resistor_SMD:R_0603_1608Metric, F.Cu at (146.0, 87.8)
- D1: value Inolux_IN-PI554FCH -> LED_Small; footprint LED_SMD:LED_Inolux_IN-PI554FCH_PLCC4_5.0x5.0mm_P3.2mm -> LED_SMD:LED_0805_2012Metric
- R1: value 1k -> 2k
- R24, R25, R26, R27, R29: value 470R -> 10k
- R35, R36, R37, R38, R39: value 5k -> 4.7k
- moved R1 5.05 mm to (148.1, 97.5), turned to 0 degrees
- moved D1 3.47 mm to (142.1, 95.3), turned to 180 degrees
- moved C26 2.45 mm to (201.4, 80.5)
- moved C27 2.45 mm to (199.3, 80.5)
- moved C28 2.45 mm to (197.1, 80.5)
- moved C29 2.45 mm to (195.0, 80.5)
Connections:
- D1 pad 1: unconnected-(D1-VSS-Pad1) -> Net-(D1-K)
- D1 pad 2: unconnected-(D1-DIN-Pad2) -> Net-(D1-A)
- R1 pad 1: LED -> +12V
- R1 pad 2: unconnected-(R1-Pad2) -> Net-(D7-A)
Routing:
- net Net-(Q8-B): track 0.00 -> 4.12 mm
- net Net-(D1-A): track 0.00 -> 2.25 mm
- net Net-(D7-A): track 0.00 -> 2.25 mm
- net Net-(D15-A1): track 232.0 -> 233.2 mm
- net Net-(D15-A2): track 228.1 -> 229.0 mm
- net +3.3V: vias 48 -> 45
- net +12V: vias 50 -> 52
- added copper zone on F.Cu, net Net-(D1-K)

Commit message: PCB layout update
Parts:
- added kibuzzard-66B57737: G***, kibuzzard-66B57737, F.Cu at (145.2, 99.8)
Routing:
- net GND: vias 763 -> 553
- net +3.3V: vias 45 -> 41

Commit message: PCB update
Parts:
- moved J11 18.4 mm to (178.1, 95.3)
- moved kibuzzard-66AC3EFD 13.4 mm to (197.6, 86.6)
- moved D4 13.4 mm to (198.7, 89.5)
- moved R20 13.4 mm to (196.2, 89.5)
- moved J2 2.76 mm to (227.1, 48.9)
- moved kibuzzard-66AC3E80 1.86 mm to (219.8, 55.5)
- moved kibuzzard-66B57737 0.25 mm to (145.0, 99.8)
Routing:
- net +3.3V: track 9.61 -> 22.3 mm, vias 41 -> 39
- net PG: track 17.9 -> 19.2 mm
- net Net-(D15-A1): track 233.2 -> 232.5 mm
- net GND: vias 553 -> 503
- added copper zone on In2.Cu, net +12V
- added copper zone on In2.Cu, net Net-(J11-Pin_1)
- removed copper zone on In1.Cu, net +12V
- removed copper zone on In1.Cu, net Net-(J11-Pin_1)
