File: HydroB V2_SubBoard/HydroB V2.kicad_sch (KiCad schematic)
At the start: 0 parts

Commit message: PCB update
Other:
- note added: "Sheet 1: Project review Sheet 2: Block of the 5 relay Sheet 3: Block of the sensor modbus Sheet 4: MCU STM32F103C8 Sheet 5: Block of Power supply the buck converter and regulator"
- note removed: "Sheet 1: Project review Sheet 2: Block of the 5 relay Sheet 3: Block of the sensor PH, EC... Sheet 4: MCU STM32F103C8 Sheet 5: Block of Power supply the buck converter and regulator Sheet 6: CANBUS TRANCEIVER"
Changed lines of the file:
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@@
 	(generator_version "8.0")
 	(paper "A4")
-	(text "Sheet 1: Project review \n\nSheet 2: Block of the 5 relay\n\nSheet 3: Block of the sensor PH, EC...\n\nSheet 4: MCU STM32F103C8\n\nSheet 5: Block of Power supply the buck converter and regulator\n\nSheet 6: CANBUS TRANCEIVER\n"
+	(text "Sheet 1: Project review \n\nSheet 2: Block of the 5 relay\n\nSheet 3: Block of the sensor modbus\n\nSheet 4: MCU STM32F103C8\n\nSheet 5: Block of Power supply the buck converter and regulator\n\n\n"
 		(exclude_from_sim no)
 		(at 19.05 56.896 0)
