File: HydroB V2_SubBoard/Power supply.kicad_sch (KiCad schematic)
At the start: 14 parts, among them U4 LMR33620ADDA

Commit message: subboard new update version
Parts:
- L2: footprint Inductor_SMD:L_7.3x7.3_H3.5 -> Inductor_SMD:L_Bourns-SRN4018
Changed lines of the file:
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@@
 			)
 		)
-		(property "Footprint" "Inductor_SMD:L_7.3x7.3_H3.5"
+		(property "Footprint" "Inductor_SMD:L_Bourns-SRN4018"
 			(at 153.67 100.33 0)
 			(effects

Commit message: PCB update
Parts:
- added J2: 12V, Connector_BarrelJack:BarrelJack_Horizontal, symbol Connector:Screw_Terminal_01x02
- L2: footprint Inductor_SMD:L_Bourns-SRN4018 -> Inductor_SMD:L_Bourns_SRP5030T
Connections:
- net +12V: now also J2.1 (Pin_1)
- net GND: now also J2.2 (Pin_2)
Other:
- moved on the sheet: C10, C23, C24, C25, C26, C27, C28, C29, C9, L2, R6, R7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
