File: HydroB V2_SubBoard/Power supply.kicad_sch (KiCad schematic)
At the start: 15 parts, among them J2 12V, U4 LMR33620ADDA

Commit message: PCB placement
Parts:
- added J11, J12: Conn_01x02_Pin, Connector_PinHeader_2.00mm:PinHeader_1x02_P2.00mm_Vertical, symbol Connector:Conn_01x02_Pin
Connections:
- net +12V: now also J11.2 (Pin_2); no longer J2.1 (Pin_1)
- net +3.3V: now also J12.2 (Pin_2); no longer C25.1, C26.1, C27.1, C28.1, C29.1, L2.2, R7.2
- new net: C25.1, C26.1, C27.1, C28.1, C29.1, J12.1 (Pin_1), L2.2, R7.2
- new net: J11.1 (Pin_1), J2.1 (Pin_1)
Other:
- moved on the sheet: J2
Changed lines of the file:
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@@
 	(wire
 		(pts
-			(xy 77.47 109.22) (xy 77.47 111.76)
+			(xy 68.58 109.22) (xy 68.58 111.76)
 		)
 		(stroke
@@
 	(wire
 		(pts
+			(xy 78.74 116.84) (xy 78.74 106.68)
+		)
+		(stroke
+			(width 0)
+			(type default)
+		)
+	)
+	(wire
+		(pts
 			(xy 208.28 129.54) (xy 198.12 129.54)
 		)
@@
 	(wire
 		(pts
+			(xy 220.98 100.33) (xy 224.79 100.33)
+		)
+		(stroke
+			(width 0)
+			(type default)
+		)
+	)
+	(wire
+		(pts
 			(xy 187.96 129.54) (xy 198.12 129.54)
 		)
@@
 	(wire
 		(pts
+			(xy 66.04 106.68) (xy 76.2 106.68)
+		)
+		(stroke
+			(width 0)
+			(type default)
+		)
+	)
+	(wire
+		(pts
+			(xy 78.74 106.68) (xy 85.09 106.68)
+		)
+		(stroke
+			(width 0)
+			(type default)
+		)
+	)
+	(wire
+		(pts
 			(xy 168.91 123.19) (xy 168.91 129.54)
 		)
@@
 	(wire
 		(pts
-			(xy 74.93 106.68) (xy 85.09 106.68)
+			(xy 76.2 106.68) (xy 76.2 116.84)
 		)
 		(stroke
@@
 	(wire
 		(pts
-			(xy 208.28 100.33) (xy 209.55 100.33)
+			(xy 208.28 100.33) (xy 218.44 100.33)
 		)
 		(stroke
@@
 	(wire
 		(pts
-			(xy 74.93 109.22) (xy 77.47 109.22)
+			(xy 66.04 109.22) (xy 68.58 109.22)
 		)
 		(stroke
@@
 	)
 	(rectangle
-		(start 58.42 74.93)
-		(end 220.98 140.97)
+		(start 46.99 74.93)
+		(end 252.73 140.97)
 		(stroke
 			(width 0)
@@
 	(symbol
 		(lib_id "power:GND")
-		(at 77.47 111.76 0)
+		(at 68.58 111.76 0)
 		(unit 1)
 		(exclude_from_sim no)
@@
 		(on_board yes)
 		(dnp no)
-		(fields_autoplaced yes)
 		(property "Reference" "#PWR02"
-			(at 77.47 118.11 0)
+			(at 68.58 118.11 0)
 			(effects
 				(font
@@
 		)
 		(property "Value" "GND"
-			(at 77.47 116.205 0)
+			(at 68.58 116.205 0)
 			(effects
 				(font
@@
 		)
 		(property "Footprint" ""
-			(at 77.47 111.76 0)
+			(at 68.58 111.76 0)
 			(effects
 				(font
@@
 		)
 		(property "Datasheet" ""
-			(at 77.47 111.76 0)
+			(at 68.58 111.76 0)
 			(effects
 				(font
@@
 		)
 		(property "Description" ""
-			(at 77.47 111.76 0)
+			(at 68.58 111.76 0)
 			(effects
 				(font
@@
 	(symbol
 		(lib_id "Connector:Screw_Terminal_01x02")
-		(at 69.85 106.68 0)
+		(at 60.96 106.68 0)
 		(mirror y)
 		(unit 1)
@@
 		(dnp no)
 		(property "Reference" "J2"
-			(at 69.85 115.57 0)
+			(at 60.96 115.57 0)
 			(effects
 				(font
@@
 		)
 		(property "Value" "12V"
-			(at 69.85 113.03 0)
+			(at 60.96 113.03 0)
 			(effects
 				(font
@@
 		)
 		(property "Footprint" "Library:DC conn"
-			(at 69.85 106.68 0)
+			(at 60.96 106.68 0)
 			(effects
 				(font
@@
 		)
 		(property "Datasheet" "~"
-			(at 69.85 106.68 0)
+			(at 60.96 106.68 0)
 			(effects
 				(font
@@
 		)
 		(property "Description" "Generic screw terminal, single row, 01x02, script generated (kicad-library-utils/schlib/autogen/connector/)"
-			(at 69.85 106.68 0)
+			(at 60.96 106.68 0)
 			(effects
 				(font
@@
 		)
 		(property "MANUFACTURER" ""
-			(at 69.85 106.68 0)
+			(at 60.96 106.68 0)
 			(effects
 				(font
@@
 		)
 		(property "MAXIMUM_PACKAGE_HEIGHT" ""
-			(at 69.85 106.68 0)
+			(at 60.96 106.68 0)
 			(effects
 				(font
@@
 		)
 		(property "PARTREV" ""
-			(at 69.85 106.68 0)
+			(at 60.96 106.68 0)
 			(effects
 				(font
@@
 		)
 		(property "STANDARD" ""
-			(at 69.85 106.68 0)
+			(at 60.96 106.68 0)
 			(effects
 				(font
@@
 		)
 		(property "Sim.Device" ""
-			(at 69.85 106.68 0)
+			(at 60.96 106.68 0)
 			(effects
 				(font
@@
 		)
 		(property "Sim.Pins" ""
-			(at 69.85 106.68 0)
+			(at 60.96 106.68 0)
 			(effects
 				(font
@@
 		)
 		(property "Sim.Type" ""
-			(at 69.85 106.68 0)
+			(at 60.96 106.68 0)
 			(effects
 				(font
@@
 	(symbol
 		(lib_id "power:+3.3V")
-		(at 209.55 100.33 270)
+		(at 224.79 100.33 270)
 		(unit 1)
 		(exclude_from_sim no)
@@
 		(fields_autoplaced yes)
 		(property "Reference" "#PWR021"
-			(at 205.74 100.33 0)
+			(at 220.98 100.33 0)
 			(effects
 				(font
@@
 		)
 		(property "Value" "+3.3V"
-			(at 213.36 100.3299 90)
+			(at 228.6 100.3299 90)
 			(effects
 				(font
@@
 		)
 		(property "Footprint" ""
-			(at 209.55 100.33 0)
+			(at 224.79 100.33 0)
 			(effects
 				(font
@@
 		)
 		(property "Datasheet" ""
-			(at 209.55 100.33 0)
+			(at 224.79 100.33 0)
 			(effects
 				(font
@@
 		)
 		(property "Description" "Power symbol creates a global label with name \"+3.3V\""
-			(at 209.55 100.33 0)
+			(at 224.79 100.33 0)
 			(effects
 				(font
@@
 	)
 	(symbol
+		(lib_id "Connector:Conn_01x02_Pin")
+		(at 76.2 121.92 90)
+		(unit 1)
+		(exclude_from_sim no)
+		(in_bom yes)
+		(on_board yes)
+		(dnp no)
+		(property "Reference" "J11"
+			(at 71.12 123.698 90)
+			(effects
+				(font
+					(size 1.27 1.27)
+				)
+				(justify right)
+			)
+		)
+		(property "Value" "Conn_01x02_Pin"
+			(at 67.564 126.238 90)
+			(effects
+				(font
+					(size 1.27 1.27)
+				)
+				(justify right)
+			)
+		)
+		(property "Footprint" "Connector_PinHeader_2.00mm:PinHeader_1x02_P2.00mm_Vertical"
+			(at 76.2 121.92 0)
+			(effects
+				(font
+					(size 1.27 1.27)
+				)
+				(hide yes)
+			)
+		)
+		(property "Datasheet" "~"
+			(at 76.2 121.92 0)
+			(effects
+				(font
+					(size 1.27 1.27)
+				)
+				(hide yes)
+			)
+		)
+		(property "Description" "Generic connector, single row, 01x02, script generated"
+			(at 76.2 121.92 0)
+			(effects
+				(font
+					(size 1.27 1.27)
+				)
+				(hide yes)
+			)
+		)
+		(pin "2"
+		)
+		(pin "1"
+		)
+		(instances
+			(project "HydroB V2"
+				(path "/0a8bb8df-6bdd-4d10-933b-144d3fa4f517/b5cea501-254b-4c6a-af47-d8c013c279ab/d50825f3-7645-4f22-8c9c-6a6002c3efba"
+					(reference "J11")
+					(unit 1)
+				)
+			)
+		)
+	)
+	(symbol
 		(lib_id "Device:C")
 		(at 158.75 109.22 0)
@@
 					(unit 1)
 				)
+			)
+		)
+	)
+	(symbol
+		(lib_id "Connector:Conn_01x02_Pin")
+		(at 218.44 105.41 90)
+		(unit 1)
+		(exclude_from_sim no)
+		(in_bom yes)
+		(on_board yes)
+		(dnp no)
+		(property "Reference" "J12"
+			(at 213.36 107.188 90)
+			(effects
+				(font
+					(size 1.27 1.27)
+				)
+				(justify right)
+			)
+		)
+		(property "Value" "Conn_01x02_Pin"
+			(at 209.804 109.728 90)
+			(effects
+				(font
+					(size 1.27 1.27)
+				)
+				(justify right)
+			)
+		)
+		(property "Footprint" "Connector_PinHeader_2.00mm:PinHeader_1x02_P2.00mm_Vertical"
+			(at 218.44 105.41 0)
+			(effects
+				(font
+					(size 1.27 1.27)
+				)
+				(hide yes)
+			)
+		)
+		(property "Datasheet" "~"
+			(at 218.44 105.41 0)
+			(effects
+				(font
+					(size 1.27 1.27)
+				)
+				(hide yes)
+			)
+		)
+		(property "Description" "Generic connector, single row, 01x02, script generated"
+			(at 218.44 105.41 0)
+			(effects
+				(font
+					(size 1.27 1.27)
+				)
+				(hide yes)
+			)
+		)
+		(pin "2"
+		)
+		(pin "1"
+		)
+		(instances
+			(project "HydroB V2"
+				(path "/0a8bb8df-6bdd-4d10-933b-144d3fa4f517/b5cea501-254b-4c6a-af47-d8c013c279ab/d50825f3-7645-4f22-8c9c-6a6002c3efba"
+					(reference "J12")
+					(unit 1)
+				)

Commit message: PCB layout
Parts:
- removed J12: Conn_01x02_Pin, Connector_PinHeader_2.00mm:PinHeader_1x02_P2.00mm_Vertical, symbol Connector:Conn_01x02_Pin
Connections:
- net +3.3V: now also C25.1, C26.1, C27.1, C28.1, C29.1, L2.2, R7.2
Changed lines of the file:
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@@
-	(wire
-		(pts
-			(xy 220.98 100.33) (xy 224.79 100.33)
-		)
-		(stroke
-			(width 0)
-			(type default)
-		)
-	)
 	(wire
 		(pts
@@
 	(wire
 		(pts
-			(xy 208.28 100.33) (xy 218.44 100.33)
+			(xy 208.28 100.33) (xy 214.63 100.33)
 		)
 		(stroke
@@
 	(rectangle
 		(start 46.99 74.93)
-		(end 252.73 140.97)
+		(end 243.84 140.97)
 		(stroke
 			(width 0)
@@
 	(symbol
 		(lib_id "power:+3.3V")
-		(at 224.79 100.33 270)
+		(at 214.63 100.33 270)
 		(unit 1)
 		(exclude_from_sim no)
@@
 		(fields_autoplaced yes)
 		(property "Reference" "#PWR021"
-			(at 220.98 100.33 0)
+			(at 210.82 100.33 0)
 			(effects
 				(font
@@
 		)
 		(property "Value" "+3.3V"
-			(at 228.6 100.3299 90)
+			(at 218.44 100.3299 90)
 			(effects
 				(font
@@
 		)
 		(property "Footprint" ""
-			(at 224.79 100.33 0)
+			(at 214.63 100.33 0)
 			(effects
 				(font
@@
 		)
 		(property "Datasheet" ""
-			(at 224.79 100.33 0)
+			(at 214.63 100.33 0)
 			(effects
 				(font
@@
 		)
 		(property "Description" "Power symbol creates a global label with name \"+3.3V\""
-			(at 224.79 100.33 0)
+			(at 214.63 100.33 0)
 			(effects
 				(font
@@
 					(unit 1)
 				)
-			)
-		)
-	)
-	(symbol
-		(lib_id "Connector:Conn_01x02_Pin")
-		(at 218.44 105.41 90)
-		(unit 1)
-		(exclude_from_sim no)
-		(in_bom yes)
-		(on_board yes)
-		(dnp no)
-		(property "Reference" "J12"
-			(at 213.36 107.188 90)
-			(effects
-				(font
-					(size 1.27 1.27)
-				)
-				(justify right)
-			)
-		)
-		(property "Value" "Conn_01x02_Pin"
-			(at 209.804 109.728 90)
-			(effects
-				(font
-					(size 1.27 1.27)
-				)
-				(justify right)
-			)
-		)
-		(property "Footprint" "Connector_PinHeader_2.00mm:PinHeader_1x02_P2.00mm_Vertical"
-			(at 218.44 105.41 0)
-			(effects
-				(font
-					(size 1.27 1.27)
-				)
-				(hide yes)
-			)
-		)
-		(property "Datasheet" "~"
-			(at 218.44 105.41 0)
-			(effects
-				(font
-					(size 1.27 1.27)
-				)
-				(hide yes)
-			)
-		)
-		(property "Description" "Generic connector, single row, 01x02, script generated"
-			(at 218.44 105.41 0)
-			(effects
-				(font
-					(size 1.27 1.27)
-				)
-				(hide yes)
-			)
-		)
-		(pin "2"
-		)
-		(pin "1"
-		)
-		(instances
-			(project "HydroB V2"
-				(path "/0a8bb8df-6bdd-4d10-933b-144d3fa4f517/b5cea501-254b-4c6a-af47-d8c013c279ab/d50825f3-7645-4f22-8c9c-6a6002c3efba"
-					(reference "J12")
-					(unit 1)
-				)
