File: HydroB V2_SubBoard/MCU.kicad_sch (KiCad schematic)
At the start: 23 parts, among them J4 Conn_01x04_Pin, SW1 SW_Push, U1 STM32F103C8Tx, Y1 8Mhz

Commit message: finish the subboard layout
Parts:
- J4: footprint Connector_JST:JST_PH_B4B-PH-K_1x04_P2.00mm_Vertical -> Connector_JST:JST_XH_B4B-XH-A_1x04_P2.50mm_Vertical
Changed lines of the file:
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@@
 			)
 		)
-		(property "Footprint" "Connector_JST:JST_PH_B4B-PH-K_1x04_P2.00mm_Vertical"
+		(property "Footprint" "Connector_JST:JST_XH_B4B-XH-A_1x04_P2.50mm_Vertical"
 			(at 44.45 105.41 0)
 			(effects

Commit message: subboard updated for PCB placement
Parts:
- SW1: footprint Button_Switch_SMD:SW_Push_SPST_NO_Alps_SKRK -> Button_Switch_SMD:SW_SPST_B3U-3000P
Changed lines of the file:
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@@
 			)
 		)
-		(property "Footprint" "Button_Switch_SMD:SW_Push_SPST_NO_Alps_SKRK"
+		(property "Footprint" "Button_Switch_SMD:SW_SPST_B3U-3000P"
 			(at 189.23 86.36 0)
 			(effects

Commit message: PCB layout update
Parts:
- SW1: footprint Button_Switch_SMD:SW_SPST_B3U-3000P -> Button_Switch_THT:SW_Tactile_SPST_Angled_PTS645Vx39-2LFS
Connections:
- net RELAY_1: now also U1.40 (PB4); no longer U1.20 (PB2)
- net RELAY_2: now also U1.41 (PB5); no longer U1.18 (PB0)
- net RELAY_3: now also U1.43 (PB7); no longer U1.46 (PB9)
- net RELAY_4: now also U1.45 (PB8); no longer U1.19 (PB1)
Changed lines of the file:
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@@
 	)
 	(no_connect
-		(at 92.71 105.41)
+		(at 92.71 95.25)
 	)
 	(no_connect
@@
 	)
 	(no_connect
-		(at 92.71 115.57)
-	)
-	(no_connect
-		(at 92.71 107.95)
+		(at 92.71 118.11)
+	)
+	(no_connect
+		(at 92.71 100.33)
 	)
 	(no_connect
@@
 	)
 	(no_connect
-		(at 92.71 113.03)
+		(at 92.71 97.79)
 	)
 	(wire
@@
 	(hierarchical_label "RELAY_2"
 		(shape input)
-		(at 92.71 95.25 180)
+		(at 92.71 107.95 180)
 		(fields_autoplaced yes)
 		(effects
@@
 	(hierarchical_label "RELAY_4"
 		(shape input)
-		(at 92.71 97.79 180)
+		(at 92.71 115.57 180)
 		(fields_autoplaced yes)
 		(effects
@@
 	(hierarchical_label "RELAY_1"
 		(shape input)
-		(at 92.71 100.33 180)
+		(at 92.71 105.41 180)
 		(fields_autoplaced yes)
 		(effects
@@
 	(hierarchical_label "RELAY_3"
 		(shape input)
-		(at 92.71 118.11 180)
+		(at 92.71 113.03 180)
 		(fields_autoplaced yes)
 		(effects
@@
 			)
 		)
-		(property "Footprint" "Button_Switch_SMD:SW_SPST_B3U-3000P"
+		(property "Footprint" "Button_Switch_THT:SW_Tactile_SPST_Angled_PTS645Vx39-2LFS"
 			(at 189.23 86.36 0)
 			(effects

Commit message: subboard new update version
Connections:
- net EN_RS485: now also U1.29 (PA8); no longer U1.11 (PA1)
- net LED: now also U1.45 (PB8); no longer U1.2 (PC13)
- net RELAY_1: now also U1.15 (PA5); no longer U1.40 (PB4)
- net RELAY_2: now also U1.13 (PA3); no longer U1.41 (PB5)
- net RELAY_3: now also U1.12 (PA2); no longer U1.43 (PB7)
- net RELAY_4: now also U1.46 (PB9); no longer U1.45 (PB8)
- net RELAY_5: now also U1.17 (PA7); no longer U1.3 (PC14)
- net RS485_RX: now also U1.31 (PA10); no longer U1.13 (PA3)
- net RS485_TX: now also U1.30 (PA9); no longer U1.12 (PA2)
- net CAN_RX: no longer names the net of U1.32 (PA11)
- net CAN_TX: no longer names the net of U1.33 (PA12)
- no-connect marks 22 -> 24
Changed lines of the file:
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@@
 	)
 	(no_connect
-		(at 125.73 115.57)
+		(at 125.73 123.19)
 	)
 	(no_connect
@@
 	)
 	(no_connect
+		(at 92.71 105.41)
+	)
+	(no_connect
+		(at 92.71 125.73)
+	)
+	(no_connect
+		(at 92.71 110.49)
+	)
+	(no_connect
+		(at 92.71 107.95)
+	)
+	(no_connect
+		(at 92.71 102.87)
+	)
+	(no_connect
+		(at 125.73 97.79)
+	)
+	(no_connect
+		(at 92.71 123.19)
+	)
+	(no_connect
+		(at 92.71 113.03)
+	)
+	(no_connect
+		(at 92.71 90.17)
+	)
+	(no_connect
+		(at 125.73 133.35)
+	)
+	(no_connect
+		(at 92.71 87.63)
+	)
+	(no_connect
 		(at 92.71 95.25)
 	)
 	(no_connect
-		(at 92.71 125.73)
-	)
-	(no_connect
-		(at 125.73 113.03)
-	)
-	(no_connect
-		(at 92.71 110.49)
-	)
-	(no_connect
-		(at 92.71 102.87)
-	)
-	(no_connect
-		(at 92.71 123.19)
-	)
-	(no_connect
-		(at 125.73 118.11)
-	)
-	(no_connect
-		(at 92.71 90.17)
-	)
-	(no_connect
-		(at 125.73 133.35)
-	)
-	(no_connect
-		(at 125.73 107.95)
-	)
-	(no_connect
 		(at 92.71 128.27)
 	)
@@
 	)
 	(no_connect
+		(at 92.71 85.09)
+	)
+	(no_connect
 		(at 92.71 130.81)
 	)
@@
 	)
 	(no_connect
-		(at 92.71 118.11)
+		(at 125.73 125.73)
 	)
 	(no_connect
 		(at 92.71 100.33)
-	)
-	(no_connect
-		(at 125.73 120.65)
 	)
 	(no_connect
@@
 	(global_label "LED"
 		(shape input)
-		(at 92.71 85.09 180)
+		(at 92.71 115.57 180)
 		(fields_autoplaced yes)
 		(effects
@@
 		)
 		(property "Intersheetrefs" "${INTERSHEET_REFS}"
-			(at 86.2777 85.09 0)
+			(at 86.2777 115.57 0)
 			(effects
 				(font
@@
 	(hierarchical_label "RS485_RX"
 		(shape input)
+		(at 125.73 120.65 0)
+		(fields_autoplaced yes)
+		(effects
+			(font
+				(size 1.27 1.27)
+			)
+			(justify left)
+		)
+	)
+	(hierarchical_label "RELAY_2"
+		(shape input)
 		(at 125.73 102.87 0)
 		(fields_autoplaced yes)
@@
 		)
 	)
-	(hierarchical_label "RELAY_2"
-		(shape input)
-		(at 92.71 107.95 180)
+	(hierarchical_label "RELAY_4"
+		(shape input)
+		(at 92.71 118.11 180)
 		(fields_autoplaced yes)
 		(effects
@@
 		)
 	)
-	(hierarchical_label "RELAY_4"
-		(shape input)
-		(at 92.71 115.57 180)
-		(fields_autoplaced yes)
-		(effects
-			(font
-				(size 1.27 1.27)
-			)
-			(justify right)
-		)
-	)
 	(hierarchical_label "EN_RS485"
 		(shape input)
-		(at 125.73 97.79 0)
+		(at 125.73 115.57 0)
 		(fields_autoplaced yes)
 		(effects
@@
 		)
 	)
-	(hierarchical_label "CAN_RX"
-		(shape input)
-		(at 125.73 123.19 0)
+	(hierarchical_label "RELAY_1"
+		(shape input)
+		(at 125.73 107.95 0)
 		(fields_autoplaced yes)
 		(effects
@@
 		)
 	)
-	(hierarchical_label "CAN_TX"
-		(shape input)
-		(at 125.73 125.73 0)
+	(hierarchical_label "RELAY_5"
+		(shape input)
+		(at 125.73 113.03 0)
 		(fields_autoplaced yes)
 		(effects
@@
 		)
 	)
-	(hierarchical_label "RELAY_1"
-		(shape input)
-		(at 92.71 105.41 180)
-		(fields_autoplaced yes)
-		(effects
-			(font
-				(size 1.27 1.27)
-			)
-			(justify right)
-		)
-	)
-	(hierarchical_label "RELAY_5"
-		(shape input)
-		(at 92.71 87.63 180)
-		(fields_autoplaced yes)
-		(effects
-			(font
-				(size 1.27 1.27)
-			)
-			(justify right)
-		)
-	)
 	(hierarchical_label "RS485_TX"
 		(shape input)
+		(at 125.73 118.11 0)
+		(fields_autoplaced yes)
+		(effects
+			(font
+				(size 1.27 1.27)
+			)
+			(justify left)
+		)
+	)
+	(hierarchical_label "RELAY_3"
+		(shape input)
 		(at 125.73 100.33 0)
 		(fields_autoplaced yes)
@@
 		)
 	)
-	(hierarchical_label "RELAY_3"
-		(shape input)
-		(at 92.71 113.03 180)
-		(fields_autoplaced yes)
-		(effects
-			(font
-				(size 1.27 1.27)
-			)
-			(justify right)
-		)
-	)

Commit message: PCB update
Parts:
- added D16, D17: LED_Small, LED_SMD:LED_0805_2012Metric, symbol Device:LED_Small
- added J5, J7: Conn_01x02_Pin, Connector_PinHeader_2.00mm:PinHeader_1x02_P2.00mm_Vertical, symbol Connector:Conn_01x02_Pin
- added Q6, Q7: S8050, Package_TO_SOT_SMD:SOT-23, symbol Transistor_BJT:S8050
- added R29, R30: 1k, Resistor_SMD:R_0603_1608Metric, symbol Device:R
- added R31, R33: 1K, Resistor_SMD:R_0603_1608Metric, symbol Device:R
- added R32, R34: 10K, Resistor_SMD:R_0603_1608Metric, symbol Device:R
- J4: footprint Connector_JST:JST_XH_B4B-XH-A_1x04_P2.50mm_Vertical -> Connector_PinHeader_2.00mm:PinHeader_1x04_P2.00mm_Vertical
Connections:
- net GND: now also D16.1 (K), D17.1 (K), Q6.2 (E), Q7.2 (E), R32.1, R34.1
- net RELAY_1: now also U1.32 (PA11); no longer U1.15 (PA5)
- net RELAY_2: now also U1.33 (PA12); no longer U1.13 (PA3)
- net RELAY_3: now also U1.38 (PA15); no longer U1.12 (PA2)
- net RELAY_4: now also U1.39 (PB3); no longer U1.46 (PB9)
- net RELAY_5: now also U1.40 (PB4); no longer U1.17 (PA7)
- net SWCLK: now also R29.1
- net SWDIO: now also R30.1
- net LED2: now reaches U1.16 (PA6)
- net LED2: now also R33.1
- new net: Q6.1 (B), R31.2, R32.2
- new net: J7.2 (Pin_2), Q7.3 (C)
- new net: Q7.1 (B), R33.2, R34.2
- new net: D16.2 (A), R29.2
- new net: J5.2 (Pin_2), Q6.3 (C)
- new net: D17.2 (A), R30.2
- new net +12V: J5.1 (Pin_1), J7.1 (Pin_1)
- new net LED1: R31.1, U1.17 (PA7)
- no-connect marks 24 -> 22
Other:
- moved on the sheet: C11, C12, C13, C14, C15, C4, C6, C7, C8, D1, D4, H5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

Commit message: new update
Connections:
- net +12V is gone; now on net +3.3V: J5.1 (Pin_1), J7.1 (Pin_1)
