File: HydroB V2_SubBoard/MCU.kicad_sch (KiCad schematic)
At the start: 31 parts, among them J4 Conn_01x04_Pin, J5 Conn_01x02_Pin, J7 Conn_01x02_Pin, Q6 S8050, Q7 S8050, SW1 SW_Push, U1 STM32F103C8Tx, Y1 8Mhz

Commit message: PCB placement
Parts:
- removed D16, D17: LED_Small, LED_SMD:LED_0805_2012Metric, symbol Device:LED_Small
- removed R29, R30: 1k, Resistor_SMD:R_0603_1608Metric, symbol Device:R
- added R17, R21: Variable Resistor, Resistor_SMD:R_0603_1608Metric, symbol Device:R
- added TP1, TP2: TestPoint, TestPoint:TestPoint_Loop_D1.80mm_Drill1.0mm_Beaded, symbol Connector:TestPoint
- C14, C15: value 22PF -> 22pF
Connections:
- net +3.3V: now also R17.1, R21.1; no longer J5.1 (Pin_1), J7.1 (Pin_1)
- net RS485_RX: now also TP2.1
- net RS485_TX: now also TP1.1
- new net: J7.1 (Pin_1), R21.2
- new net: J5.1 (Pin_1), R17.2

Commit message: PCB placement
Parts:
- removed D1: LED_Small, LED_SMD:LED_Cree-PLCC4_5x5mm_CW, symbol Device:LED_Small
- added D1: Inolux_IN-PI554FCH, LED_SMD:LED_Inolux_IN-PI554FCH_PLCC4_5.0x5.0mm_P3.2mm, symbol LED:Inolux_IN-PI554FCH
Other:
- moved on the sheet: R1
Changed lines of the file:
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@@
 	(wire
 		(pts
-			(xy 73.66 133.35) (xy 77.47 133.35)
-		)
-		(stroke
-			(width 0)
-			(type default)
-		)
-	)
-	(wire
-		(pts
 			(xy 93.98 163.83) (xy 96.52 163.83)
 		)
@@
 	(wire
 		(pts
-			(xy 53.34 133.35) (xy 55.88 133.35)
+			(xy 45.72 128.27) (xy 48.26 128.27)
 		)
 		(stroke
@@
 	(wire
 		(pts
-			(xy 63.5 133.35) (xy 68.58 133.35)
-		)
-		(stroke
-			(width 0)
-			(type default)
-		)
-	)
-	(wire
-		(pts
 			(xy 110.49 138.43) (xy 113.03 138.43)
 		)
@@
 	(global_label "LED"
 		(shape input)
-		(at 53.34 133.35 180)
+		(at 45.72 128.27 180)
 		(fields_autoplaced yes)
 		(effects
@@
 		)
 		(property "Intersheetrefs" "${INTERSHEET_REFS}"
-			(at 46.9077 133.35 0)
+			(at 39.2877 128.27 0)
 			(effects
 				(font
@@
 	(symbol
 		(lib_id "Device:R")
-		(at 59.69 133.35 90)
+		(at 52.07 128.27 90)
 		(unit 1)
 		(exclude_from_sim no)
@@
 		(fields_autoplaced yes)
 		(property "Reference" "R1"
-			(at 59.69 127 90)
+			(at 52.07 121.92 90)
 			(effects
 				(font
@@
 		)
 		(property "Value" "1k"
-			(at 59.69 129.54 90)
+			(at 52.07 124.46 90)
 			(effects
 				(font
@@
 		)
 		(property "Footprint" "Resistor_SMD:R_0603_1608Metric"
-			(at 59.69 135.128 90)
+			(at 52.07 130.048 90)
 			(effects
 				(font
@@
 		)
 		(property "Datasheet" "~"
-			(at 59.69 133.35 0)
+			(at 52.07 128.27 0)
 			(effects
 				(font
@@
 		)
 		(property "Description" "Resistor"
-			(at 59.69 133.35 0)
+			(at 52.07 128.27 0)
 			(effects
 				(font
@@
 	)
 	(symbol
-		(lib_id "Device:LED_Small")
-		(at 71.12 133.35 180)
-		(unit 1)
-		(exclude_from_sim no)
-		(in_bom yes)
-		(on_board yes)
-		(dnp no)
-		(fields_autoplaced yes)
-		(property "Reference" "D1"
-			(at 71.0565 127 0)
-			(effects
-				(font
-					(size 1.27 1.27)
-				)
-			)
-		)
-		(property "Value" "LED_Small"
-			(at 71.0565 129.54 0)
-			(effects
-				(font
-					(size 1.27 1.27)
-				)
-			)
-		)
-		(property "Footprint" "LED_SMD:LED_Cree-PLCC4_5x5mm_CW"
-			(at 71.12 133.35 90)
-			(effects
-				(font
-					(size 1.27 1.27)
-				)
-				(hide yes)
-			)
-		)
-		(property "Datasheet" "~"
-			(at 71.12 133.35 90)
-			(effects
-				(font
-					(size 1.27 1.27)
-				)
-				(hide yes)
-			)
-		)
-		(property "Description" "Light emitting diode, small symbol"
-			(at 71.12 133.35 0)
-			(effects
-				(font
-					(size 1.27 1.27)
-				)
-				(hide yes)
-			)
-		)
-		(pin "1"
-		)
-		(pin "2"
-		)
-		(instances
-			(project "HydroB V2"
-				(path "/0a8bb8df-6bdd-4d10-933b-144d3fa4f517/b5cea501-254b-4c6a-af47-d8c013c279ab/ec9ee8ef-fc9d-4925-9304-49bf7b4d5612"
-					(reference "D1")
-					(unit 1)
-				)
-			)
-		)
-	)
-	(symbol
 		(lib_id "Connector:TestPoint")
 		(at 149.86 95.25 0)
@@
 	)
 	(symbol
+		(lib_id "LED:Inolux_IN-PI554FCH")
+		(at 68.58 127 0)
+		(unit 1)
+		(exclude_from_sim no)
+		(in_bom yes)
+		(on_board yes)
+		(dnp no)
+		(property "Reference" "D1"
+			(at 79.502 118.11 0)
+			(effects
+				(font
+					(size 1.27 1.27)
+				)
+			)
+		)
+		(property "Value" "Inolux_IN-PI554FCH"
+			(at 79.502 120.65 0)
+			(effects
+				(font
+					(size 1.27 1.27)
+				)
+			)
+		)
+		(property "Footprint" "LED_SMD:LED_Inolux_IN-PI554FCH_PLCC4_5.0x5.0mm_P3.2mm"
+			(at 69.85 134.62 0)
+			(effects
+				(font
+					(size 1.27 1.27)
+				)
+				(justify left top)
+				(hide yes)
+			)
+		)
+		(property "Datasheet" "http://www.inolux-corp.com/datasheet/SMDLED/Addressable%20LED/IN-PI554FCH.pdf"
+			(at 71.12 136.525 0)
+			(effects
+				(font
+					(size 1.27 1.27)
+				)
+				(justify left top)
+				(hide yes)
+			)
+		)
+		(property "Description" "5050 RGB LED 4-Pin with integrated IC"
+			(at 68.58 127 0)
+			(effects
+				(font
+					(size 1.27 1.27)
+				)
+				(hide yes)
+			)
+		)
+		(pin "3"
+		)
+		(pin "1"
+		)
+		(pin "2"
+		)
+		(pin "4"
+		)
+		(instances
+			(project "HydroB V2"
+				(path "/0a8bb8df-6bdd-4d10-933b-144d3fa4f517/b5cea501-254b-4c6a-af47-d8c013c279ab/ec9ee8ef-fc9d-4925-9304-49bf7b4d5612"
+					(reference "D1")
+					(unit 1)
+				)
+			)
+		)
+	)
+	(symbol
 		(lib_id "Device:C_Small")
 		(at 204.47 133.35 0)
@@
 					(unit 1)
 				)
-			)
-		)
-	)
-	(symbol
-		(lib_name "GND_1")
-		(lib_id "power:GND")
-		(at 77.47 133.35 90)
-		(unit 1)
-		(exclude_from_sim no)
-		(in_bom yes)
-		(on_board yes)
-		(dnp no)
-		(fields_autoplaced yes)
-		(property "Reference" "#PWR01"
-			(at 83.82 133.35 0)
-			(effects
-				(font
-					(size 1.27 1.27)
-				)
-				(hide yes)
-			)
-		)
-		(property "Value" "GND"
-			(at 81.28 133.3499 90)
-			(effects
-				(font
-					(size 1.27 1.27)
-				)
-				(justify right)
-			)
-		)
-		(property "Footprint" ""
-			(at 77.47 133.35 0)
-			(effects
-				(font
-					(size 1.27 1.27)
-				)
-				(hide yes)
-			)
-		)
-		(property "Datasheet" ""
-			(at 77.47 133.35 0)
-			(effects
-				(font
-					(size 1.27 1.27)
-				)
-				(hide yes)
-			)
-		)
-		(property "Description" "Power symbol creates a global label with name \"GND\" , ground"
-			(at 77.47 133.35 0)
-			(effects
-				(font
-					(size 1.27 1.27)
-				)
-				(hide yes)
-			)
-		)
-		(pin "1"
-		)
-		(instances
-			(project "HydroB V2"
-				(path "/0a8bb8df-6bdd-4d10-933b-144d3fa4f517/b5cea501-254b-4c6a-af47-d8c013c279ab/ec9ee8ef-fc9d-4925-9304-49bf7b4d5612"
-					(reference "#PWR01")
-					(unit 1)
-				)

Commit message: PCB layout
Connections:
- net EN_RS485: now also U1.11 (PA1); no longer U1.14 (PA4)
- net LED1: now also U1.18 (PB0); no longer U1.30 (PA9)
- net LED2: now also U1.21 (PB10); no longer U1.32 (PA11)
- net RELAY_1: now also U1.39 (PB3); no longer U1.46 (PB9)
- net RELAY_2: now also U1.41 (PB5); no longer U1.45 (PB8)
- net RELAY_3: now also U1.42 (PB6); no longer U1.43 (PB7)
- net RELAY_4: now also U1.45 (PB8); no longer U1.41 (PB5)
- net RELAY_5: now also U1.46 (PB9); no longer U1.42 (PB6)

Commit message: update
Parts:
- removed D1: Inolux_IN-PI554FCH, LED_SMD:LED_Inolux_IN-PI554FCH_PLCC4_5.0x5.0mm_P3.2mm, symbol LED:Inolux_IN-PI554FCH
- added D1, D7: LED_Small, LED_SMD:LED_0805_2012Metric, symbol Device:LED_Small
- added Q8: S8050, Package_TO_SOT_SMD:SOT-23, symbol Transistor_BJT:S8050
- added R18: 10K, Resistor_SMD:R_0603_1608Metric, symbol Device:R
- added R2: 2k, Resistor_SMD:R_0603_1608Metric, symbol Device:R
- added R3: 1K, Resistor_SMD:R_0603_1608Metric, symbol Device:R
- R1: value 1k -> 2k
Connections:
- net GND: now also Q8.2 (E), R18.1
- net LED: now also R3.1; no longer R1.1
- net at R1.2: now also D7.2 (A)
- new net: Q8.1 (B), R18.2, R3.2
- new net: D1.1 (K), D7.1 (K), Q8.3 (C)
- new net: D1.2 (A), R2.2
- new net +12V: R1.1, R2.1
Other:
- moved on the sheet: D4, J4, R20

Commit message: PCB update
Other:
- note added: "LED INDICATOR"
- moved on the sheet: C11, C12, C13, C14, C15, C4, C6, C7, C8, D1, D4, D7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
