File: HydroB V2_SubBoard/Block Sensor.kicad_sch (KiCad schematic)
At the start: 8 parts, among them J5 PH SENSOR, J6 EC SENSOR, U3 SN65HVD72DR

Commit message: finish the subboard layout
Parts:
- J5, J6: footprint Connector_Phoenix_MC:PhoenixContact_MCV_1,5_4-G-3.81_1x04_P3.81mm_Vertical -> Connector_Phoenix_MC:PhoenixContact_MC_1,5_4-G-3.81_1x04_P3.81mm_Horizontal
Changed lines of the file:
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@@
 			)
 		)
-		(property "Footprint" "Connector_Phoenix_MC:PhoenixContact_MCV_1,5_4-G-3.81_1x04_P3.81mm_Vertical"
+		(property "Footprint" "Connector_Phoenix_MC:PhoenixContact_MC_1,5_4-G-3.81_1x04_P3.81mm_Horizontal"
 			(at 156.21 105.41 0)
 			(effects
@@
 			)
 		)
-		(property "Footprint" "Connector_Phoenix_MC:PhoenixContact_MCV_1,5_4-G-3.81_1x04_P3.81mm_Vertical"
+		(property "Footprint" "Connector_Phoenix_MC:PhoenixContact_MC_1,5_4-G-3.81_1x04_P3.81mm_Horizontal"
 			(at 171.45 105.41 0)
 			(effects

Commit message: subboard updated for PCB placement
Parts:
- J5, J6: footprint Connector_Phoenix_MC:PhoenixContact_MC_1,5_4-G-3.81_1x04_P3.81mm_Horizontal -> Connector_Phoenix_MC:PhoenixContact_MCV_1,5_4-G-3.81_1x04_P3.81mm_Vertical
Connections:
- net +24V renamed +12V
Changed lines of the file:
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@@
+	)
+	(symbol
+		(lib_id "power:+12V")
+		(at 161.29 85.09 0)
+		(unit 1)
+		(exclude_from_sim no)
+		(in_bom yes)
+		(on_board yes)
+		(dnp no)
+		(fields_autoplaced yes)
+		(property "Reference" "#PWR055"
+			(at 161.29 88.9 0)
+			(effects
+				(font
+					(size 1.27 1.27)
+				)
+				(hide yes)
+			)
+		)
+		(property "Value" "+12V"
+			(at 161.29 80.01 0)
+			(effects
+				(font
+					(size 1.27 1.27)
+				)
+			)
+		)
+		(property "Footprint" ""
+			(at 161.29 85.09 0)
+			(effects
+				(font
+					(size 1.27 1.27)
+				)
+				(hide yes)
+			)
+		)
+		(property "Datasheet" ""
+			(at 161.29 85.09 0)
+			(effects
+				(font
+					(size 1.27 1.27)
+				)
+				(hide yes)
+			)
+		)
+		(property "Description" "Power symbol creates a global label with name \"+12V\""
+			(at 161.29 85.09 0)
+			(effects
+				(font
+					(size 1.27 1.27)
+				)
+				(hide yes)
+			)
+		)
+		(pin "1"
+		)
+		(instances
+			(project "HydroB V2"
+				(path "/0a8bb8df-6bdd-4d10-933b-144d3fa4f517/b5cea501-254b-4c6a-af47-d8c013c279ab/8f835ad3-c2cc-4f7e-9766-2e7525ceefc9"
+					(reference "#PWR055")
+					(unit 1)
+				)
+			)
+		)
 	)
 	(symbol
@@
 	)
 	(symbol
-		(lib_id "power:+24V")
-		(at 161.29 85.09 0)
-		(unit 1)
-		(exclude_from_sim no)
-		(in_bom yes)
-		(on_board yes)
-		(dnp no)
-		(fields_autoplaced yes)
-		(property "Reference" "#PWR02"
-			(at 161.29 88.9 0)
-			(effects
-				(font
-					(size 1.27 1.27)
-				)
-				(hide yes)
-			)
-		)
-		(property "Value" "+24V"
-			(at 161.29 80.01 0)
-			(effects
-				(font
-					(size 1.27 1.27)
-				)
-			)
-		)
-		(property "Footprint" ""
-			(at 161.29 85.09 0)
-			(effects
-				(font
-					(size 1.27 1.27)
-				)
-				(hide yes)
-			)
-		)
-		(property "Datasheet" ""
-			(at 161.29 85.09 0)
-			(effects
-				(font
-					(size 1.27 1.27)
-				)
-				(hide yes)
-			)
-		)
-		(property "Description" "Power symbol creates a global label with name \"+24V\""
-			(at 161.29 85.09 0)
-			(effects
-				(font
-					(size 1.27 1.27)
-				)
-				(hide yes)
-			)
-		)
-		(pin "1"
-		)
-		(instances
-			(project "HydroB V2"
-				(path "/0a8bb8df-6bdd-4d10-933b-144d3fa4f517/b5cea501-254b-4c6a-af47-d8c013c279ab/8f835ad3-c2cc-4f7e-9766-2e7525ceefc9"
-					(reference "#PWR02")
-					(unit 1)
-				)
-			)
-		)
-	)
-	(symbol
 		(lib_id "Connector:Conn_01x04_Pin")
 		(at 156.21 105.41 90)
@@
 			)
 		)
-		(property "Footprint" "Connector_Phoenix_MC:PhoenixContact_MC_1,5_4-G-3.81_1x04_P3.81mm_Horizontal"
+		(property "Footprint" "Connector_Phoenix_MC:PhoenixContact_MCV_1,5_4-G-3.81_1x04_P3.81mm_Vertical"
 			(at 156.21 105.41 0)
 			(effects
@@
 			)
 		)
-		(property "Footprint" "Connector_Phoenix_MC:PhoenixContact_MC_1,5_4-G-3.81_1x04_P3.81mm_Horizontal"
+		(property "Footprint" "Connector_Phoenix_MC:PhoenixContact_MCV_1,5_4-G-3.81_1x04_P3.81mm_Vertical"
 			(at 171.45 105.41 0)
 			(effects

Commit message: subboard new update version
Parts:
- added D7, D8: LED_Small, LED_SMD:LED_0805_2012Metric, symbol Device:LED_Small
- added R17, R21: 10k, Resistor_SMD:R_0603_1608Metric, symbol Device:R
Connections:
- net +3.3V: now also D7.2 (A), D8.2 (A)
- net RS485_RX: now also R21.1
- net RS485_TX: now also R17.1
- new net: D7.1 (K), R21.2
- new net: D8.1 (K), R17.2
Other:
- moved on the sheet: J6, R15

Commit message: PCB update
Parts:
- removed J5: PH SENSOR, Connector_Phoenix_MC:PhoenixContact_MCV_1,5_4-G-3.81_1x04_P3.81mm_Vertical, symbol Connector:Conn_01x04_Pin
- added D15: D_TVS, Diode_SMD:D_SOD-123F, symbol Device:D_TVS
- added J1: Conn_01x02_Pin, Connector_Phoenix_MC:PhoenixContact_MCV_1,5_2-G-3.81_1x02_P3.81mm_Vertical, symbol Connector:Conn_01x02_Pin
- J6: value EC SENSOR -> SENSOR
Connections:
- net at J6.2 (Pin_2), R10.2, R15.1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: now also D15.1 (A1), J1.1 (Pin_1)
- net at J6.3 (Pin_3), R15.2, R4.1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: now also D15.2 (A2), J1.2 (Pin_2)
Other:
- moved on the sheet: J6, R15

Commit message: PCB component placement and layout
Parts:
- J1: footprint Connector_Phoenix_MC:PhoenixContact_MCV_1,5_2-G-3.81_1x02_P3.81mm_Vertical -> hydroB:Din sensor
- J6: footprint Connector_Phoenix_MC:PhoenixContact_MCV_1,5_4-G-3.81_1x04_P3.81mm_Vertical -> hydroB:Din sensor 4 Pin
Changed lines of the file:
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@@
 			)
 		)
-		(property "Footprint" "Connector_Phoenix_MC:PhoenixContact_MCV_1,5_2-G-3.81_1x02_P3.81mm_Vertical"
+		(property "Footprint" "hydroB:Din sensor"
 			(at 171.45 111.76 0)
 			(effects
@@
 			)
 		)
-		(property "Footprint" "Connector_Phoenix_MC:PhoenixContact_MCV_1,5_4-G-3.81_1x04_P3.81mm_Vertical"
+		(property "Footprint" "hydroB:Din sensor 4 Pin"
 			(at 184.15 113.03 0)
 			(effects

Commit message: PCB placement
Parts:
- removed D7, D8: LED_Small, LED_SMD:LED_0805_2012Metric, symbol Device:LED_Small
- removed R17, R21: 10k, Resistor_SMD:R_0603_1608Metric, symbol Device:R
- added TP3, TP4: TestPoint, TestPoint:TestPoint_Loop_D1.80mm_Drill1.0mm_Beaded, symbol Connector:TestPoint
Connections:
- net at D15.1 (A1), J1.1 (Pin_1), J6.2 (Pin_2)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: now also TP4.1
- net at D15.2 (A2), J1.2 (Pin_2), J6.3 (Pin_3)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: now also TP3.1
Other:
- moved on the sheet: J1, J6

Commit message: PCB layout
Changed lines of the file:
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@@
 	)
 	(rectangle
-		(start 63.5 54.102)
+		(start 87.63 54.102)
 		(end 210.82 135.89)
 		(stroke
