File: HydroB V2_SubBoard/Block Relay.kicad_sch (KiCad schematic)
At the start: 50 parts, among them J10 Screw_Terminal_01x02, J16 Screw_Terminal_01x02, J3 Screw_Terminal_01x02, J8 Screw_Terminal_01x02, J9 Screw_Terminal_01x02, Q1 S8050, Q2 S8050, Q3 S8050, Q4 S8050, Q5 S8050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

Commit message: PCB placement
Parts:
- removed R18, R2, R22, R23, R3: 10K, Resistor_SMD:R_0603_1608Metric, symbol Device:R
- R24, R25, R26, R27, R29: value 445R -> 470R
- R35, R36, R37, R38, R39: value 220R -> 5k
Connections:
- net +3.3V is gone; now on net GND: R24.1, R25.1, R26.1, R29.1

Commit message: update
Parts:
- R24, R25, R26, R27, R29: value 470R -> 10k
- R35, R36, R37, R38, R39: value 5k -> 4.7k
Changed lines of the file:
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@@
 			)
 		)
-		(property "Value" "5k"
-			(at 27.94 41.91 90)
+		(property "Value" "4.7k"
+			(at 27.178 41.91 90)
 			(effects
 				(font
@@
 			)
 		)
-		(property "Value" "470R"
+		(property "Value" "10k"
 			(at 118.11 88.9 90)
 			(effects
@@
 			)
 		)
-		(property "Value" "470R"
+		(property "Value" "10k"
 			(at 257.81 35.56 90)
 			(effects
@@
 			)
 		)
-		(property "Value" "5k"
-			(at 28.194 152.4 90)
+		(property "Value" "4.7k"
+			(at 26.924 152.654 90)
 			(effects
 				(font
@@
 			)
 		)
-		(property "Value" "470R"
+		(property "Value" "10k"
 			(at 115.57 35.56 90)
 			(effects
@@
 			)
 		)
-		(property "Value" "5k"
-			(at 165.1 95.25 90)
+		(property "Value" "4.7k"
+			(at 164.084 95.25 90)
 			(effects
 				(font
@@
 			)
 		)
-		(property "Value" "470R"
+		(property "Value" "10k"
 			(at 257.81 91.44 90)
 			(effects
@@
 			)
 		)
-		(property "Value" "5k"
-			(at 27.94 95.25 90)
+		(property "Value" "4.7k"
+			(at 26.924 95.25 90)
 			(effects
 				(font
@@
 			)
 		)
-		(property "Value" "470R"
-			(at 118.11 148.59 90)
+		(property "Value" "10k"
+			(at 117.348 148.59 90)
 			(effects
 				(font
@@
 			)
 		)
-		(property "Value" "5k"
-			(at 166.624 40.64 90)
+		(property "Value" "4.7k"
+			(at 165.354 40.64 90)
 			(effects
 				(font
