File: HydroB V2.kicad_pcb (KiCad board)
At the start: 4 copper layers, 180.2 x 120 mm, 133 parts, among them J1 Conn_01x02_Pin, J10 Screw_Terminal_01x02, J11 Conn_01x02_Pin, J16 Screw_Terminal_01x02, J2 12V, J3 Screw_Terminal_01x02, J4 Conn_01x04_Pin, J5 Conn_01x02_Pin, J6 SENSOR, J7 Conn_01x02_Pin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

Commit message: Updated label
Parts:
- removed the kibuzzard-66AB40EF at (97.3, 35.4)
- removed the kibuzzard-66AB40EF at (75.5, 35.4)
- removed the kibuzzard-66AB40EF at (141.1, 35.4)
- removed the kibuzzard-66AB40EF at (119.2, 35.4)
- removed the kibuzzard-66AB40EF at (163.0, 35.4)
- removed kibuzzard-66AB4112 (x5): G***, kibuzzard-66AB4112
- removed kibuzzard-66B57737: G***, kibuzzard-66B57737
- added kibuzzard-66B9A896: G***, kibuzzard-66B9A896, F.Cu at (73.0, 35.4)
- added kibuzzard-66B9A89E: G***, kibuzzard-66B9A89E, F.Cu at (75.5, 35.4)
- added kibuzzard-66B9A8C9: G***, kibuzzard-66B9A8C9, F.Cu at (94.7, 35.4)
- added kibuzzard-66B9A8CF: G***, kibuzzard-66B9A8CF, F.Cu at (97.2, 35.4)
- added kibuzzard-66B9A8D4: G***, kibuzzard-66B9A8D4, F.Cu at (116.7, 35.4)
- added kibuzzard-66B9A8DE: G***, kibuzzard-66B9A8DE, F.Cu at (119.2, 35.4)
- added kibuzzard-66B9A8E4: G***, kibuzzard-66B9A8E4, F.Cu at (138.6, 35.4)
- added kibuzzard-66B9A8E9: G***, kibuzzard-66B9A8E9, F.Cu at (141.1, 35.4)
- added kibuzzard-66B9A8EF: G***, kibuzzard-66B9A8EF, F.Cu at (160.5, 35.4)
- added kibuzzard-66B9A8F6: G***, kibuzzard-66B9A8F6, F.Cu at (163.0, 35.4)
- added kibuzzard-66B9A932: G***, kibuzzard-66B9A932, F.Cu at (195.2, 75.5)
- moved kibuzzard-66AC3E80 2.33 mm to (221.1, 57.4)
- moved kibuzzard-66AC3E8A 0.20 mm to (226.5, 90.5)
- moved kibuzzard-66AC3EE5 0.18 mm to (222.0, 73.7)
